File: _autosave-Hard-EnvSens.kicad_sch (KiCad schematic)
At the start: 49 parts, among them P1 USB_C_Plug_USB2.0, P2 USB_C_Plug_USB2.0, Q1 SS8050, Q2 SS8050, SW1 SW_Push, SW3 SW_Push, U1 LD1117S33TR_SOT223, U2 ESP32-C6-WROOM-1, U3 CP2104, U4 VEML7700-TR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

Commit message: Dps368
Parts:
- removed U5: DPS310, DPS310:XDCR_DPS310, symbol DPS310:DPS310
- added C18, C19: 100nF, symbol Device:C_Small
- added D4: LED, symbol Device:LED
- added R13: 4.7k, symbol Device:R
- added U5: DPS368, DPS368:LGA8S145X65P2X4_200X250X110-V, symbol DPS368:DPS368
Connections:
- net GND: now also C18.2, C19.2, D4.1 (K), U5.1 (GND_1), U5.7 (GND_2)
- net Scl: now also U5.4 (SCK)
- net Sda: now also U5.3 (SDI)
- net at U2.23 (GPIO15): now also R13.2
- new net: C18.1, C19.1, U5.6 (VDDIO), U5.8 (VDD)
- new net: D4.2 (A), R13.1
Other:
- note added: "Debug USB"
- moved on the sheet: C1, C2, C3, D3, P2, Q1, Q2, R1, R17, R18, R19, R2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
