File: Hard-EnvSens.kicad_pcb (KiCad board)
At the start: 2 copper layers, 60 x 75.6 mm, 59 parts, among them J1 TYPE-C-31-M-12, J2 Conn_01x04_Socket, J3 Conn_02x02_Odd_Even, J4 Conn_01x04_Pin, J5 Conn_02x02_Odd_Even, Q1 SS8050, Q2 SS8050, SW1 SW_Push, SW3 SW_Push, U1 LD1117S33TR_SOT223, U2 ESP32-C6-WROOM-1, U4 VEML7700-TR, U5 DPS368, U6 SGP41-D-R4, U7 SHT40-AD1B-R2, U8 AS7341-DLGT, U9 TPS79318DBVTG4

Commit message: Baterry charger + giroscope
Magnetometer not connected
Parts:
- added C10: 22uF, Capacitor_SMD:C_0603_1608Metric, F.Cu at (66.4, 77.8)
- added C25: 22uF, Capacitor_SMD:C_0603_1608Metric, F.Cu at (66.4, 80.3)
- added C26: 22uF, Capacitor_SMD:C_0603_1608Metric, F.Cu at (119.4, 78.2)
- added C27: 22uF, Capacitor_SMD:C_0603_1608Metric, F.Cu at (119.4, 79.8)
- added C28: 10uF, Capacitor_SMD:C_0603_1608Metric, F.Cu at (119.4, 75.0)
- added C29: 10uF, Capacitor_SMD:C_0603_1608Metric, F.Cu at (119.4, 71.8)
- added C8: 22uF, Capacitor_SMD:C_0603_1608Metric, F.Cu at (127.0, 71.8)
- added C9: 22uF, Capacitor_SMD:C_0603_1608Metric, F.Cu at (127.0, 70.3)
- added D3: LED, LED_SMD:LED_0603_1608Metric, F.Cu at (102.9, 72.2)
- added J6: Conn_01x02_Pin, Connector_PinHeader_2.54mm:PinHeader_1x02_P2.54mm_Vertical, F.Cu at (103.2, 65.7)
- added L1: 1uH, Inductor_SMD:L_TechFuse_SL0630, F.Cu at (109.5, 67.2)
- added R15: 2R, Resistor_SMD:R_0603_1608Metric, F.Cu at (119.4, 73.4)
- added R16: 0.5R, Resistor_SMD:R_0603_1608Metric, F.Cu at (119.4, 76.6)
- added R20: 100k, Resistor_SMD:R_0603_1608Metric, F.Cu at (123.8, 79.0)
- added R21: 10k, Resistor_SMD:R_0603_1608Metric, F.Cu at (127.0, 79.0)
- added SW2: SW_Push, Biblioteca_Kicad:SW_3-1437565-0, F.Cu at (71.3, 67.8)
- added U3: IP5306, libs:SOP127P600X165-9N, F.Cu at (124.8, 75.4)
- moved C4 21.3 mm to (129.4, 71.0)
- moved U1 14.4 mm to (128.3, 65.8)
- moved C11 9.22 mm to (127.6, 59.3), turned to 180 degrees
- moved D1 7.21 mm to (122.3, 52.7)
- moved R10 7.21 mm to (122.3, 54.7)
- moved R13 7.21 mm to (125.9, 54.7)
- moved D4 7.21 mm to (125.9, 52.7)
- moved C5 6.97 mm to (127.6, 60.9), turned to 180 degrees
- moved C1 3.30 mm to (151.3, 65.6)
- moved C2 3.30 mm to (151.3, 64.0)
- moved R2 1.00 mm to (138.6, 68.7)
- moved C3 0.32 mm to (131.4, 60.9), turned to 180 degrees
- moved R8 0.22 mm to (131.4, 59.3), turned to 0 degrees
- moved J3 0.10 mm to (146.9, 117.8)
Connections:
- net +5V renamed +5vBat
Routing:
- net +3V3: track 155.4 -> 88.2 mm
- net Net-(U2-GPIO15): track 48.1 -> 23.8 mm
- net EN: track 27.8 -> 17.1 mm
- net +5vBat: track 22.3 -> 11.9 mm
- net GND: track 63.7 -> 61.6 mm, vias 31 -> 30
- net Net-(U2-GPIO8): track 2.55 -> 3.57 mm

Commit message: Correct commit for battery charger
Parts:
- added C30: 100nF, Capacitor_SMD:C_0603_1608Metric, F.Cu at (112.7, 92.9)
- added C31: 100nF, Capacitor_SMD:C_0603_1608Metric, F.Cu at (112.7, 94.5)
- added C32: 100nF, Capacitor_SMD:C_0603_1608Metric, F.Cu at (112.7, 96.5)
- added C33: 100nF, Capacitor_SMD:C_0603_1608Metric, F.Cu at (112.7, 98.2)
- added D5: SS14, Diode_SMD:D_SMA, F.Cu at (122.1, 74.5)
- added D6: SS14, Diode_SMD:D_SMA, F.Cu at (107.5, 67.2)
- added R22: 4.7k, Resistor_SMD:R_0603_1608Metric, F.Cu at (105.5, 94.8)
- added R23: 4.7k, Resistor_SMD:R_0603_1608Metric, F.Cu at (103.8, 94.8)
- added U10: BMI160, Package_LGA:Bosch_LGA-14_3x2.5mm_P0.5mm, F.Cu at (109.2, 93.8)
- added U11: BMM150, Package_CSP:WLCSP-12_1.56x1.56mm_P0.4mm, F.Cu at (109.0, 97.1)
- moved C25 55.0 mm to (118.5, 62.8)
- moved C10 53.8 mm to (118.5, 64.3)
- moved SW2 39.0 mm to (108.8, 57.2), turned to -90 degrees
- moved C9 13.9 mm to (115.4, 62.8)
- moved C8 13.9 mm to (115.4, 64.3)
- moved L1 12.8 mm to (117.6, 57.4), turned to 180 degrees
- moved R15 12.4 mm to (110.1, 65.2), turned to -90 degrees
- moved R20 12.3 mm to (114.1, 71.7)
- moved R21 12.3 mm to (117.2, 71.7)
- moved C26 11.3 mm to (110.9, 70.8)
- moved C28 11.3 mm to (110.9, 67.6)
- moved U3 11.3 mm to (116.3, 68.0)
- moved C27 11.3 mm to (110.9, 72.5)
- moved R16 11.3 mm to (110.8, 69.3)
- moved C29 10.2 mm to (111.7, 65.2), turned to 90 degrees
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Connections:
- C28 pad 1: +5vBat -> +5V
- C4 pad 1: +5vBat -> Net-(D5-K)
- D2 pad 4: +5vBat -> +5V
- J1 pad A4_B9: +5vBat -> +5V
- J1 pad B4_A9: +5vBat -> +5V
- R15 pad 1: +5vBat -> +5V
- U1 pad 3: +5vBat -> Net-(D5-K)
- U2 pad 16: unconnected-(U2-GPIO18-Pad16) -> Int1
- U3 pad 1: +5vBat -> +5V
Routing:
- net +3V3: track 88.2 -> 169.2 mm
- net Net-(J6-Pin_2): track 0.00 -> 31.9 mm
- net Net-(D5-K): track 0.00 -> 27.7 mm
- net +5V: track 0.00 -> 24.4 mm
- net GND: track 61.6 -> 80.1 mm, vias 30 -> 49
- net Net-(U2-GPIO15): track 23.8 -> 42.0 mm
- net Sda: track 24.6 -> 39.0 mm, vias 0 -> 1
- net Scl: track 29.3 -> 42.9 mm, vias 0 -> 1
- net Net-(D3-A): track 0.00 -> 12.7 mm, vias 0 -> 2
- net Net-(U3-BAT): track 0.00 -> 11.4 mm
- net Net-(U3-SW): track 0.00 -> 10.5 mm, vias 0 -> 4
- net EN: track 17.1 -> 27.4 mm
- net Net-(U10-ASCx): track 0.00 -> 7.07 mm
- net Net-(U3-LED2): track 0.00 -> 6.79 mm, vias 0 -> 2
- net +5vBat: track 11.9 -> 18.3 mm
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- added copper zone on B.Cu, net (none)
- added copper zone on F.Cu, net (none)
- added copper zone on B.Cu, net Net-(U3-SW)

Commit message: Improved whole board design
Parts:
- removed C33: 100nF, Capacitor_SMD:C_0603_1608Metric
- removed R22, R23: 4.7k, Resistor_SMD:R_0603_1608Metric
- removed U11: BMM150, Package_CSP:WLCSP-12_1.56x1.56mm_P0.4mm
- Gas: renamed from U6; footprint Biblioteca_Kicad:XDCR_SGP41-D-R4 -> libs:XDCR_SGP41-D-R4
- Humidity: renamed from U7; footprint Biblioteca_Kicad:SHT4X -> libs:SHT4X
- J1: footprint Biblioteca_Kicad:HRO_TYPE-C-31-M-12 -> libs:HRO_TYPE-C-31-M-12
- J3, J4: moved to B.Cu
- Light: renamed from U4; footprint Biblioteca_Kicad:XDCR_VEML7700-TR -> libs:XDCR_VEML7700-TR
- R13: value 4.7k -> 1k
- R21: value 10k -> 1k
- SW1, SW2, SW3: footprint Biblioteca_Kicad:SW_3-1437565-0 -> libs:Botao KH-6X6X5H-STM
- U2: footprint PCM_Espressif:ESP32-C6-WROOM-1 -> libs:XCVR_ESP32-C6-WROOM-1-N8
- moved C32 52.9 mm to (120.1, 44.2)
- moved SW2 11.3 mm to (107.7, 45.9), turned to 0 degrees
- moved J2 6.01 mm to (111.8, 98.3)
- moved J5 6.00 mm to (140.2, 100.9)
- moved R21 3.49 mm to (114.1, 73.2), turned to 0 degrees
- moved U2 3.01 mm to (146.6, 79.9)
- moved J3 1.46 mm to (146.4, 116.5), turned to 180 degrees
- moved SW1 0.65 mm to (148.6, 54.5)
- moved SW3 0.63 mm to (135.8, 54.6)
- moved J4 0.40 mm to (117.8, 113.9), turned to 180 degrees
- moved C12 0.32 mm to (124.3, 119.9)
- moved C13 0.32 mm to (125.9, 119.9)
- moved R9 0.32 mm to (122.7, 119.9)
- moved C29 0.12 mm to (111.8, 65.2)
- renumbered U8 to Colour, MK1 to Mic, U5 to Pressure, R20 to R20*1
Connections:
- C32 pad 1: +3V3 -> Net-(U3-KEY)
- J3 pad 2: SCKtop -> SDtop
- J3 pad 3: SDtop -> SCKtop
- R21 pad 1: Net-(U3-KEY) -> Net-(U3-LED3)
- R21 pad 2: Net-(R21-Pad2) -> Net-(U3-BAT)
- SW1 pad 4: (no net) -> GND
- SW2 pad 2: Net-(R21-Pad2) -> Net-(U3-KEY)
- SW3 pad 4: (no net) -> GND
- U10 pad 2: Net-(U10-ASDx) -> unconnected-(U10-ASDx-Pad2)
- U10 pad 3: Net-(U10-ASCx) -> unconnected-(U10-ASCx-Pad3)
- U3 pad 4: Net-(U3-LED2) -> Net-(U3-LED3)
Routing:
- net Int1: track 0.00 -> 38.2 mm, vias 0 -> 2
- net +3V3: track 169.2 -> 134.5 mm, vias 0 -> 19
- net GND: track 80.1 -> 68.1 mm, vias 49 -> 126
- net +5V: track 24.4 -> 33.8 mm, vias 0 -> 16
- net Net-(U10-ASCx): track 7.07 -> 0.00 mm
- net Net-(U3-LED3): track 0.00 -> 6.94 mm, vias 0 -> 2
- net +1V8: track 32.7 -> 26.7 mm
- net Net-(U2-GPIO0/ADC1_CH0/XTAL_32K_P): track 20.4 -> 25.6 mm
- net Net-(U10-ASDx): track 4.94 -> 0.00 mm
- net Scl: track 42.9 -> 47.0 mm
- net IO9: track 24.2 -> 27.8 mm
- net EN: track 27.4 -> 30.8 mm
- net Sda: track 39.0 -> 42.1 mm
- net WS: track 30.5 -> 33.4 mm
- net SD: track 31.0 -> 33.7 mm
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- added copper zone on B.Cu, net +3V3
- added copper zone on F.Cu, net +3V3
- added copper zone on B.Cu, net +5V
- added copper zone on F.Cu, net +5V
Other:
- outline, holes or cut-outs redrawn

Commit message: Lot of improvements
Parts:
- J6: footprint Connector_PinHeader_2.54mm:PinHeader_1x02_P2.54mm_Vertical -> Connector_Molex:Molex_KK-254_AE-6410-02A_1x02_P2.54mm_Vertical
- moved ON 56.5 mm to (147.7, 103.9)
- moved Status 52.2 mm to (147.6, 100.9)
- moved BOOST 51.9 mm to (104.2, 97.7), turned to 90 degrees
- moved R10 43.1 mm to (145.1, 92.1), turned to -90 degrees
- moved R13 42.1 mm to (146.7, 92.1), turned to 90 degrees
- moved C32 25.8 mm to (121.8, 70.0), turned to -90 degrees
- moved C18 6.07 mm to (131.9, 114.1)
- moved MK1 6.07 mm to (132.4, 123.6)
- moved C16 6.07 mm to (135.9, 114.1)
- moved U5 6.07 mm to (128.9, 114.7)
- moved U7 6.07 mm to (137.9, 113.5)
- moved C12 6.07 mm to (118.3, 120.9)
- moved C13 6.07 mm to (119.9, 120.9)
- moved C14 6.07 mm to (121.5, 116.8)
- moved C15 6.07 mm to (116.7, 116.8)
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- renumbered U9 to 1.8V, U1 to 3V3, SW2 to BOOST, SW3 to ENABLE, U2 to ESP32-C6-WROOM, Mic to MK1, D1 to ON, R20*1 to R20, D4 to Status, Light to U4, Pressure to U5, Gas to U6, Humidity to U7, Colour to U8, J1 to USB-C
Connections:
- BOOST pad 3: (no net) -> Net-(U3-KEY)
- BOOST pad 4: (no net) -> GND
- ENABLE pad 4: GND -> (no net)
- SW1 pad 4: GND -> (no net)
Routing:
- net Net-(U2-GPIO15): track 43.8 -> 3.46 mm, vias 2 -> 0
- net Net-(U3-KEY): track 0.01 -> 40.2 mm, vias 0 -> 2
- net GND: track 68.1 -> 48.6 mm, vias 126 -> 150
- net Net-(D1-A): track 2.02 -> 13.9 mm
- net Net-(D4-A): track 2.01 -> 11.4 mm
- net +5V: track 33.8 -> 41.9 mm, vias 16 -> 15
- net Net-(U3-SW): track 10.5 -> 2.98 mm, vias 4 -> 8
- net +3V3: track 134.5 -> 129.5 mm, vias 19 -> 21
- net Int1: track 38.2 -> 42.3 mm
- net +1V8: track 26.7 -> 23.4 mm, vias 1 -> 3
- net Net-(J6-Pin_2): track 29.2 -> 32.6 mm
- net EN: track 30.8 -> 33.1 mm
- net Net-(U3-LED3): track 6.94 -> 4.67 mm
- net Sda: track 42.1 -> 44.2 mm
- net Scl: track 47.0 -> 48.7 mm
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- added copper zone on B.Cu, net +1V8
- added copper zone on F.Cu, net +1V8
- added copper zone on F.Cu, net GND2
- added copper zone on F.Cu, net Net-(J6-Pin_2)
- added copper zone on F.Cu, net Net-(U3-SW)
Other:
- board size 60 x 75.6 mm -> 60 x 76.6 mm
- board text added: "+"
- board text added: "-"

Commit message: Logos and corrections
Parts:
- added G***: LOGO, Images:hanze, F.Cu at (153.8, 63.7)
- added G***: LOGO, Images:fapes, F.Cu at (157.9, 63.6)
- added G***: LOGO, Images:2solve, F.Cu at (153.8, 97.4)
- added G***: LOGO, Images:labtel, F.Cu at (157.6, 97.5)
- moved C1 4.08 mm to (147.9, 63.4), turned to -90 degrees
- moved C2 1.99 mm to (149.5, 63.4), turned to -90 degrees
- moved D3 1.39 mm to (106.1, 72.9), turned to 0 degrees
- moved ON 0.62 mm to (147.6, 104.5)
- moved 3V3 0.22 mm to (128.2, 67.3)
Routing:
- net GND: track 48.6 -> 42.9 mm, vias 150 -> 162
- net Net-(D1-A): track 13.9 -> 14.5 mm
- net Net-(U3-SW): vias 8 -> 12
- net (no net): vias 0 -> 4
Other:
- outline, holes or cut-outs redrawn
- board text added: "Battery"
