File: Hard-EnvSens.kicad_pcb (KiCad board)
At the start: 2 copper layers, 60 x 77.7 mm, 111 parts, among them J1 TYPE-C-31-M-12, J2 Conn_01x04_Socket, J3 Conn_02x02_Odd_Even, J4 Conn_01x04_Pin, J5 Conn_02x02_Odd_Even, J6 Conn_01x02_Pin, J7 Conn_01x04_Pin, Q1 SS8050, Q2 SS8050, U10 BMI160, U11 TPS22918TDBVRQ1, U12*1 TP4056-42-ESOP8, U13 SPX3819M5-L-3-3, U2 ESP32-C6-WROOM-1, U3 IP5306, U4 VEML7700-TR, U5 DPS368, U6 SGP41-D-R4, U7 SHT40-AD1B-R2, U8 AS7341-DLGT, U9 TPS79318DBVTG4

Commit message: Upgrading the product
Parts:
- removed ? (x3): , 
- removed C11: 100nF, Capacitor_SMD:C_0603_1608Metric
- removed REF**: Hole 3mm, libs:Hole 3mm
- SW2: renamed from ON / OFF
- moved C5 24.8 mm to (151.2, 69.5), turned to 0 degrees
- moved C1 5.63 mm to (151.2, 68.0), turned to 0 degrees
- moved C2 3.55 mm to (151.2, 66.5), turned to 0 degrees
- moved R6 0.10 mm to (145.4, 63.8)
- renumbered Sensor to 3V3Sensor1, Boost to 5vBoost1, Usb to 5vUSB1, Bat to Battery1, GND to GND1, J7 to J7*1, MIC to MK1, R20 to R20*1, R30 to R30*1, RX to RX1, BOOT to SW1, Enable to SW3, TX to TX1
Connections:
- U2 pad 29_1: GND -> (no net)
- U2 pad 29_2: GND -> (no net)
- U2 pad 29_3: GND -> (no net)
- U2 pad 29_4: GND -> (no net)
- U2 pad 29_5: GND -> (no net)
- U2 pad 29_6: GND -> (no net)
- U2 pad 29_7: GND -> (no net)
- U2 pad 29_8: GND -> (no net)
- U2 pad 29_9: GND -> (no net)
Routing:
- net GND: track 30.6 -> 35.3 mm, vias 272 -> 273

Commit message: Comecando nova versao, muita coisa diferente
Parts:
- J1: footprint libs:HRO_TYPE-C-31-M-12 -> EnvSens:HRO_TYPE-C-31-M-12
- SW1, SW2, SW3: footprint libs:Botao KH-6X6X5H-STM -> EnvSens:Botao KH-6X6X5H-STM
- U11: footprint libs:SOT95P280X145-6N -> EnvSens:SOT95P280X145-6N
- U2: footprint libs:XCVR_ESP32-C6-WROOM-1-N8 -> EnvSens:XCVR_ESP32-C6-WROOM-1-N8
- U3: footprint libs:SOP127P600X165-9N -> EnvSens:SOP127P600X165-9N
- U4: footprint libs:XDCR_VEML7700-TR -> EnvSens:XDCR_VEML7700-TR
- U5: footprint libs:LGA8S145X65P2X4_200X250X110-V -> EnvSens:LGA8S145X65P2X4_200X250X110-V
- U6: footprint libs:XDCR_SGP41-D-R4 -> EnvSens:XDCR_SGP41-D-R4
- U7: footprint libs:SHT4X -> EnvSens:SHT4X
- U9: footprint libs:SOT95P280X145-5N -> EnvSens:SOT95P280X145-5N
Changed lines of the file:
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@@
 		)
 	)
-	(footprint "libs:XCVR_ESP32-C6-WROOM-1-N8"
+	(footprint "EnvSens:XCVR_ESP32-C6-WROOM-1-N8"
 		(layer "F.Cu")
 		(at 146.61 79.935 -90)
@@
 		)
 	)
-	(footprint "libs:XDCR_VEML7700-TR"
+	(footprint "EnvSens:XDCR_VEML7700-TR"
 		(layer "F.Cu")
 		(at 111.317 126.07 90)
@@
 		)
 	)
-	(footprint "libs:SOT95P280X145-6N"
+	(footprint "EnvSens:SOT95P280X145-6N"
 		(layer "F.Cu")
 		(at 128.33 82.7 -90)
@@
 		(embedded_fonts no)
 	)
-	(footprint "libs:Botao KH-6X6X5H-STM"
+	(footprint "EnvSens:Botao KH-6X6X5H-STM"
 		(layer "F.Cu")
 		(at 145.86 54.43 180)
@@
 		)
 	)
-	(footprint "libs:Botao KH-6X6X5H-STM"
+	(footprint "EnvSens:Botao KH-6X6X5H-STM"
 		(layer "F.Cu")
 		(at 104.06 97.74 90)
@@
 		)
 	)
-	(footprint "libs:SOP127P600X165-9N"
+	(footprint "EnvSens:SOP127P600X165-9N"
 		(layer "F.Cu")
 		(at 117.2 68.01)
@@
 		)
 	)
-	(footprint "libs:LGA8S145X65P2X4_200X250X110-V"
+	(footprint "EnvSens:LGA8S145X65P2X4_200X250X110-V"
 		(layer "F.Cu")
 		(at 120.717 115.77 90)
@@
 		)
 	)
-	(footprint "libs:SOT95P280X145-5N"
+	(footprint "EnvSens:SOT95P280X145-5N"
 		(layer "F.Cu")
 		(at 122.485 90.07)
@@
 		)
 	)
-	(footprint "libs:HRO_TYPE-C-31-M-12"
+	(footprint "EnvSens:HRO_TYPE-C-31-M-12"
 		(layer "F.Cu")
 		(at 103.1 79.7 -90)
@@
 		)
 	)
-	(footprint "libs:SHT4X"
+	(footprint "EnvSens:SHT4X"
 		(layer "F.Cu")
 		(at 129.717 114.57 -90)
@@
 		)
 	)
-	(footprint "libs:XDCR_SGP41-D-R4"
+	(footprint "EnvSens:XDCR_SGP41-D-R4"
 		(layer "F.Cu")
 		(at 111.267 114.37)
@@
 		)
 	)
-	(footprint "libs:Botao KH-6X6X5H-STM"
+	(footprint "EnvSens:Botao KH-6X6X5H-STM"
 		(layer "F.Cu")
 		(at 132.11 54.49 180)
