File: Hard-EnvSens.kicad_sch (KiCad schematic)
At the start: 101 parts, among them J1 TYPE-C-31-M-12, J2 Conn_01x04_Socket, J3 Conn_02x02_Odd_Even, J4 Conn_01x04_Pin, J5 Conn_02x02_Odd_Even, J6 Conn_01x02_Pin, J7*1 Conn_01x04_Pin, Q1 SS8050, Q2 SS8050, SW1 SW_Push, SW2 SW_Push, SW3 SW_Push, U10 BMI160, U11 TPS22918TDBVRQ1, U12*1 TP4056-42-ESOP8, U13 SPX3819M5-L-3-3, U2 ESP32-C6-WROOM-1, U3 IP5306, U4 VEML7700-TR, U5 DPS368, U6 SGP41-D-R4, U7 SHT40-AD1B-R2, U8 AS7341-DLGT, U9 TPS79318DBVTG4

Commit message: Comecando nova versao, muita coisa diferente
Parts:
- removed 1V8, 3V3, 3V3Sensor1, 5vBoost1, Battery1: TestPoint, TestPoint:TestPoint_THTPad_1.5x1.5mm_Drill0.7mm, symbol Connector:TestPoint
- removed C20, C34, C40: 0.1uF, Capacitor_SMD:C_0603_1608Metric, symbol Device:C_Small
- removed C21: 0.01uF, Capacitor_SMD:C_0603_1608Metric, symbol Device:C_Small
- removed C22, C28, C29, C36*1, C4: 10uF, Capacitor_SMD:C_0603_1608Metric, symbol Device:C_Small
- removed C23, C32: 100nF, Capacitor_SMD:C_0603_1608Metric, symbol Device:C_Small
- removed C24: 4.7uF, Capacitor_SMD:C_0603_1608Metric, symbol Device:C_Small
- removed C25, C26, C27: 22uF, Capacitor_SMD:C_0603_1608Metric, symbol Device:C_Small
- removed C33: 1uF, Capacitor_SMD:C_0603_1608Metric, symbol Device:C_Small
- removed C35: 1nF, Capacitor_SMD:C_0603_1608Metric, symbol Device:C_Small
- removed C38: 10nF, Capacitor_SMD:C_0603_1608Metric, symbol Device:C_Small
- removed C39: 100uF, Capacitor_SMD:C_Elec_6.3x7.7, symbol Device:C_Small
- removed D3: LED, LED_SMD:LED_0603_1608Metric, symbol Device:LED
- removed D5, D6, D7: CMS30I30A, Diode_SMD:D_SMA, symbol Diode:SS14
- removed J6: Conn_01x02_Pin, Connector_Molex:Molex_KK-254_AE-6410-02A_1x02_P2.54mm_Vertical, symbol Connector:Conn_01x02_Pin
- removed L1: 1uH, Inductor_SMD:L_TechFuse_SL0630, symbol Device:L
- removed MK1: ICS-43434, Sensor_Audio:InvenSense_ICS-43434-6_3.5x2.65mm, symbol Sensor_Audio:ICS-43434
- removed R15: 2R, Resistor_SMD:R_0603_1608Metric, symbol Device:R
- removed R16: 0.5R, Resistor_SMD:R_0603_1608Metric, symbol Device:R
- removed R20*1: 100k, Resistor_SMD:R_0603_1608Metric, symbol Device:R
- removed R21: 1k, Resistor_SMD:R_0603_1608Metric, symbol Device:R
- removed R30*1: 0R, Resistor_SMD:R_0603_1608Metric, symbol Device:R
- removed R31*1: 4k, Resistor_SMD:R_0603_1608Metric, symbol Device:R
- removed R32*1: 10k, Resistor_SMD:R_0603_1608Metric, symbol Device:R
- removed R7: 100K, Resistor_SMD:R_0603_1608Metric, symbol Device:R
- removed SW2: SW_Push, libs:Botao KH-6X6X5H-STM, symbol Switch:SW_Push
- removed U11: TPS22918TDBVRQ1, libs:SOT95P280X145-6N, symbol TPS22918TDBVRQ1:TPS22918TDBVRQ1
- removed U12*1: TP4056-42-ESOP8, Package_SO:SOIC-8-1EP_3.9x4.9mm_P1.27mm_EP2.41x3.3mm_ThermalVias, symbol Battery_Management:TP4056-42-ESOP8
- removed U13: SPX3819M5-L-3-3, Package_TO_SOT_SMD:SOT-23-5, symbol Regulator_Linear:SPX3819M5-L-3-3
- removed U3: IP5306, libs:SOP127P600X165-9N, symbol IP5306:IP5306
- removed U5: DPS368, libs:LGA8S145X65P2X4_200X250X110-V, symbol DPS368:DPS368
- removed U8: AS7341-DLGT, Package_LGA:AMS_OLGA-8_2x3.1mm_P0.8mm, symbol AS7341-DLGT:AS7341-DLGT
- removed U9: TPS79318DBVTG4, libs:SOT95P280X145-5N, symbol TPS793-18:TPS79318DBVTG4
- added 3V1: TestPoint, TestPoint:TestPoint_THTPad_1.5x1.5mm_Drill0.7mm, symbol Connector:TestPoint
- added C11: 22uF, Capacitor_SMD:C_0603_1608Metric, symbol Device:C_Small
- added C5: 10uF, Capacitor_SMD:C_0603_1608Metric, symbol Device:C_Small
- added D1: LED, LED_SMD:LED_0603_1608Metric, symbol Device:LED
- added D3: CMS30I30A, Diode_SMD:D_SMA, symbol Diode:SS14
- added MK1: T5838, EnvSens:MIC_T5838, symbol EnvSens:T5838
- added Q3: AO3401A, Package_TO_SOT_SMD:SOT-23, symbol Transistor_FET:AO3401A
- added R10: 2k, symbol Device:R_Small
- added R7: 470, symbol Device:R_Small
- added U1: ESP32-S31-WROOM-1-N16R16V, EnvSens:ESP32-S31-WROOM-1, symbol EnvSens:ESP32-S31-WROOM-1-N16R16V
- added U5: MCP73831-2-OT, Package_TO_SOT_SMD:SOT-23-5, symbol Battery_Management:MCP73831-2-OT
- added U8: XC6220B331MR, Package_TO_SOT_SMD:SOT-23-5, symbol Regulator_Linear:XC6220B331MR
- C10: value 22uF -> 10uF
- C18: value 100nF -> 22uF
- C19: value 100nF -> 0.1uF
- C6: value 4.7uF -> 100uF; footprint Capacitor_SMD:C_0603_1608Metric -> Capacitor_SMD:C_Elec_6.3x7.7
- C8, C9: value 22uF -> 4.7uF
- J1: footprint libs:HRO_TYPE-C-31-M-12 -> EnvSens:HRO_TYPE-C-31-M-12; symbol TYPE-C-31-M-12:TYPE-C-31-M-12 -> EnvSens:TYPE-C-31-M-12
- R14: value 10k -> 100k
- SW1, SW3: footprint libs:Botao KH-6X6X5H-STM -> EnvSens:Botao KH-6X6X5H-STM
- U2: footprint libs:XCVR_ESP32-C6-WROOM-1-N8 -> EnvSens:XCVR_ESP32-C6-WROOM-1-N8
- U4: footprint libs:XDCR_VEML7700-TR -> EnvSens:XDCR_VEML7700-TR; symbol VEML7700-TR:VEML7700-TR -> EnvSens:VEML7700-TR
- U6: footprint libs:XDCR_SGP41-D-R4 -> EnvSens:XDCR_SGP41-D-R4; symbol SGP41-D-R4:SGP41-D-R4 -> EnvSens:SGP41-D-R4
- U7: footprint libs:SHT4X -> EnvSens:SHT4X; symbol SHT40-AD1B-R2:SHT40-AD1B-R2 -> EnvSens:SHT40-AD1B-R2
Connections:
- net +1V8top: no longer R14.2
- net +3V3: now also C18.1, C19.1, C6.1, 3V1.1, C11.1, C5.1, U1.2 (3V3), U8.5 (VOUT)
- net +3V3top: no longer C18.1, C19.1, C6.1
- net +5V: now also C8.2, R14.2, D1.2 (A), D3.2 (A), Q3.1 (G), U5.4 (V_{DD})
- net Bat+: now also C9.2, Q3.3 (D), U5.3 (V_{BAT})
- net D+: now also U1.55 (DP)
- net D-: now also U1.54 (DM)
- net GND: now also C18.2, C19.2, C6.2, C8.1, C9.1, R14.1, C11.2, C5.2, MK1.3_1 (GND), MK1.3_2 (GND), R10.1, U1.1 (GND), U1.40 (GND), U1.41 (GND), U5.2 (V_{SS}), U8.2 (GND); no longer C8.2, C9.2
- net GND2: no longer C18.2, C19.2, C6.2
- removed net +5vBat: C10.1, C8.1, C9.1
- new net: D1.1 (K), R7.1
- new net: R7.2, U5.1 (STAT)
- new net: R10.2, U5.5 (PROG)
- new net +Vin: C10.1, D3.1 (K), Q3.2 (S), U8.1 (VIN), U8.3 (CE)
- no-connect marks 19 -> 14
Other:
- note added: "3V3 LDO"
- note added: "Bat Charger"
- note removed: "*use if IP5306 isnt working"
- note removed: "2nd option for Battery charging + Power Supply"
- note removed: "3V3 to 1V8"
- note removed: "3V3/1V8"
- note removed: "5V to 3V3"
- note removed: "AS7341"
- note removed: "Battery charger + Power Supply"
- note removed: "DPS368"
- note removed: "MIC ICS-43434"
- moved on the sheet: C1, C12, C13, C14, C15, C16, C17, C2, C3, C30, C31, C7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
